Commit message: [Tilted quadrotor] implemented SR-inverse Fully actuated control

File: robots/mini_quadrotor/urdf/dual/robot.urdf.xacro (robot description, xacro)
@@ -138,6 +138,6 @@
       </visual>
   </link>
-  <joint name="flex_joint1" type="revolute">
-  <!-- <joint name="flex_joint1" type="fixed"> -->
+  <!-- <joint name="flex_joint1" type="revolute"> -->
+  <joint name="flex_joint1" type="fixed">
     <parent link="main_body1"/>
     <child link="flex_link"/>

Commit message: [URDF] modified model to have a 2dof joint in the middle

File: robots/mini_quadrotor/urdf/dual/robot.urdf.xacro (robot description, xacro)
@@ -119,7 +119,7 @@
     </collision>
   </link>
-  <link name="flex_link">
-    <inertial>
-      <origin xyz="${-flex_link_length/2} 0 0" rpy="0 ${pi/2} 0"/>
+  <link name="flex_link1">
+    <inertial>
+      <origin xyz="${-flex_link_length/8} 0 0" rpy="0 ${pi/2} 0"/>
       <mass value="0.05"/>
       <inertia
@@ -129,7 +129,7 @@
     </inertial>
       <visual>
-        <origin xyz="${-flex_link_length/2} 0 0" rpy="0 ${pi/2} 0"/>
+        <origin xyz="${-flex_link_length/4} 0 0" rpy="0 ${pi/2} 0"/>
         <geometry>
-          <cylinder length="${flex_link_length}" radius="0.03"/>
+          <cylinder length="${flex_link_length/2}" radius="0.03"/>
         </geometry>
         <material name="green">
@@ -138,8 +138,37 @@
       </visual>
   </link>
+  <link name="dummy_flex_link">
+    <inertial>
+      <origin xyz="0.000001 0 0" rpy="0 0 0"/>
+      <mass value="0.05"/>
+      <inertia
+          ixx="0.000001" ixy="0.0" ixz="0.0"
+          iyy="0.000001" iyz="0.0"
+          izz="0.000002"/>
+    </inertial>
+  </link>
+  <link name="flex_link2">
+    <inertial>
+      <origin xyz="${-flex_link_length/8} 0 0" rpy="0 ${pi/2} 0"/>
+      <mass value="0.05"/>
+      <inertia
+          ixx="0.000001" ixy="0.0" ixz="0.0"
+          iyy="0.000001" iyz="0.0"
+          izz="0.000002"/>
+    </inertial>
+      <visual>
+        <origin xyz="${-flex_link_length/4} 0 0" rpy="0 ${pi/2} 0"/>
+        <geometry>
+          <cylinder length="${flex_link_length/2}" radius="0.03"/>
+        </geometry>
+        <material name="green">
+          <color rgba="0.0 1.0 0.0 2.0"/>
+        </material>
+      </visual>
+  </link>
   <!-- <joint name="flex_joint1" type="revolute"> -->
-  <joint name="flex_joint1" type="fixed">
+  <joint name="body_joint1" type="fixed">
     <parent link="main_body1"/>
-    <child link="flex_link"/>
+    <child link="flex_link1"/>
     <origin rpy="0 0 0" xyz="0 0 ${-flex_joint_offset_z}"/>
     <axis xyz="1 0 0"/>
@@ -147,4 +176,27 @@
     <dynamics damping="0.1" friction="0.0"/>
   </joint>
+  <joint name="flex_joint_p" type="revolute">
+    <parent link="flex_link1"/>
+    <child link="dummy_flex_link"/>
+    <origin rpy="0 0 0" xyz="${-flex_link_length/2} 0 0"/>
+    <axis xyz="0 1 0"/>
+    <limit effort="0.001" lower="${-pi/2}" upper="${pi/2}" velocity="1"/>
+    <dynamics damping="0.1" friction="0.0"/>
+  </joint>
+  <gazebo reference='flex_joint_p'>
+    <springReference>0</springReference>
+    <springStiffness>2</springStiffness>
+  </gazebo>
+  <joint name="flex_joint_y" type="revolute">
+    <parent link="dummy_flex_link"/>
+    <child link="flex_link2"/>
+    <axis xyz="0 0 1"/>
+    <limit effort="0.001" lower="${-pi/2}" upper="${pi/2}" velocity="1"/>
+    <dynamics damping="0.1" friction="0.0"/>
+  </joint>
+  <gazebo reference='flex_joint_y'>
+    <springReference>0</springReference>
+    <springStiffness>2</springStiffness>
+  </gazebo>
   <!-- main_body2 -->
   <link name="main_body2">
@@ -170,8 +222,8 @@
     </collision>
   </link>
-  <joint name="flex_joint2" type="fixed">
-    <parent link="flex_link"/>
+  <joint name="body_joint2" type="fixed">
+    <parent link="flex_link2"/>
     <child link="main_body2"/>
-    <origin rpy="0 0 0" xyz="${-flex_link_length} 0 ${flex_joint_offset_z}"/>
+    <origin rpy="0 0 0" xyz="${-flex_link_length/2} 0 ${flex_joint_offset_z}"/>
     <axis xyz="1 0 0"/>
   </joint>

Commit message: [Model] tf of quadrotor2 will now be published

File: robots/mini_quadrotor/urdf/dual/robot.urdf.xacro (robot description, xacro)
@@ -186,5 +186,5 @@
   <gazebo reference='flex_joint_p'>
     <springReference>0</springReference>
-    <springStiffness>2</springStiffness>
+    <springStiffness>10</springStiffness>
   </gazebo>
   <joint name="flex_joint_y" type="revolute">
@@ -197,5 +197,5 @@
   <gazebo reference='flex_joint_y'>
     <springReference>0</springReference>
-    <springStiffness>2</springStiffness>
+    <springStiffness>10</springStiffness>
   </gazebo>
   <!-- main_body2 -->
@@ -283,3 +283,21 @@
   <xacro:propeller_module id = "7" x = "${rotor_x}" y = "${rotor_y}" z = "${rotor_z}" direction = "1" tilt = "${rotor_tilt}" par_link = "main_body2"/>
   <xacro:propeller_module id = "8" x = "${-rotor_x}" y = "${rotor_y}" z = "${rotor_z}"  direction = "-1" tilt = "${rotor_tilt}" par_link = "main_body2"/>
+  <transmission name="joint_y">
+    <type>transmission_interface/SimpleTransmission</type>
+    <actuator name="motor1">
+      <mechanicalReduction>1</mechanicalReduction>
+    </actuator>
+    <joint name="flex_joint_y">
+      <hardwareInterface>hardware_interface/EffortJointInterface</hardwareInterface>
+    </joint>
+  </transmission>
+  <transmission name="joint_p">
+    <type>transmission_interface/SimpleTransmission</type>
+    <actuator name="motor2">
+      <mechanicalReduction>1</mechanicalReduction>
+    </actuator>
+    <joint name="flex_joint_p">
+      <hardwareInterface>hardware_interface/EffortJointInterface</hardwareInterface>
+    </joint>
+  </transmission>
 </robot>

Commit message: [Control] Implemented bending control

File: robots/mini_quadrotor/urdf/dual/robot.urdf.xacro (robot description, xacro)
@@ -186,5 +186,5 @@
   <gazebo reference='flex_joint_p'>
     <springReference>0</springReference>
-    <springStiffness>10</springStiffness>
+    <springStiffness>0.8</springStiffness>
   </gazebo>
   <joint name="flex_joint_y" type="revolute">
@@ -197,5 +197,5 @@
   <gazebo reference='flex_joint_y'>
     <springReference>0</springReference>
-    <springStiffness>10</springStiffness>
+    <springStiffness>0.5</springStiffness>
   </gazebo>
   <!-- main_body2 -->
@@ -239,39 +239,4 @@
     </inertial>
   </xacro:extra_module>
-  <!-- <!-\- front realsense t265 -\-> -->
-  <!-- <xacro:extra_module name = "realsense_t265" parent = "main_body" visible = "1" scale= "1" -->
-  <!--                     model_url = "package://mini_quadrotor/urdf/mesh/realSense_t265.STL"> -->
-  <!--   <origin xyz="0.1095 0.00775 0.0125" rpy="0 0 0"/> -->
-  <!--   <inertial> -->
-  <!--     <mass value = "0.07" /> -->
-  <!--     <origin xyz="-0.007 -0.007 0" rpy="0 0 0"/> -->
-  <!--     <inertia -->
-  <!--         ixx="0.0" ixy="0.0" ixz="0.0" -->
-  <!--         iyy="0.0001" iyz="0.0" -->
-  <!--         izz="0.0001"/> -->
-  <!--   </inertial> -->
-  <!-- </xacro:extra_module> -->
-  <!-- <!-\- pose frame for realsense t265 -\-> -->
-  <!-- <xacro:extra_module name = "realsense_pose_frame" parent = "realsense_t265" visible = "0" > -->
-  <!--   <origin xyz="-0.005 0.0 0.0" rpy="0 0 0"/> -->
-  <!--   <inertial> -->
-  <!--     <mass value = "0.0" /> -->
-  <!--     <origin xyz="0 0 0" rpy="0 0 0"/> -->
-  <!--     <inertia -->
-  <!--         ixx="0.0" ixy="0.0" ixz="0.0" -->
-  <!--         iyy="0.0" iyz="0.0" izz="0.0"/> -->
-  <!--   </inertial> -->
-  <!-- </xacro:extra_module> -->
-  <!-- <!-\- battery -\-> -->
-  <!-- <xacro:extra_module name = "battery" parent = "main_body" visible = "1" model_url = "package://mini_quadrotor/urdf/mesh/turnigy_3S_2200mAh.dae" > -->
-  <!--   <origin xyz="0.0105 0 -0.012" rpy="0 0 0"/> -->
-  <!--   <inertial> -->
-  <!--     <mass value = "0.188" /> -->
-  <!--     <origin xyz="0 0 0" rpy="0 0 0"/> -->
-  <!--     <inertia -->
-  <!--         ixx="0.0" ixy="0.0" ixz="0.0" -->
-  <!--         iyy="0.0002" iyz="0.0" izz="0.0002"/> -->
-  <!--   </inertial> -->
-  <!-- </xacro:extra_module> -->
   <!-- propellers -->
   <xacro:propeller_module id = "1" x = "${-rotor_x}" y = "${-rotor_y}" z = "${rotor_z}" direction = "1" tilt = "${-rotor_tilt}" par_link = "main_body1"/>
