Commit message: updated FC location

File: robots/assemble_quadrotors/urdf/tilted/dual/robot1.urdf.xacro (robot description, xacro)
@@ -128,5 +128,5 @@
   <!-- spinal -->
   <xacro:extra_module name = "fc" parent = "main_body" visible = "0" >
-    <origin xyz="-0.22 0.0 0.0165" rpy="0 0 0"/>
+    <origin xyz="-0.613 0.0 0.0195" rpy="0 0 0"/>
     <inertial>
       <mass value = "0.05" />

File: robots/assemble_quadrotors/urdf/tilted/dual/robot2.urdf.xacro (robot description, xacro)
@@ -128,5 +128,5 @@
   <!-- spinal -->
   <xacro:extra_module name = "fc" parent = "main_body" visible = "0" >
-    <origin xyz="-0.22 0.0 0.0165" rpy="0 0 0"/>
+    <origin xyz="-0.613 0.0 0.0195" rpy="0 0 3.14159265358979"/>
     <inertial>
       <mass value = "0.05" />

Commit message: [tilted_quadrotor] Updated urdf files

File: robots/assemble_quadrotors/urdf/tilted/dual/robot1.urdf.xacro (robot description, xacro)
@@ -105,8 +105,8 @@
   <link name="main_body">
     <inertial>
-      <mass value = "1.086" />
+      <mass value = "1.586" />
       <origin xyz="0 0 0.00907" rpy="0 0 0"/>
       <inertia
-          ixx="0.0777" ixy="0.00178" ixz="0.00000"
+          ixx="0.00777" ixy="0.000178" ixz="0"
           iyy="0.407" iyz="0"
           izz="0.412"/>

File: robots/assemble_quadrotors/urdf/tilted/dual/robot2.urdf.xacro (robot description, xacro)
@@ -105,8 +105,8 @@
   <link name="main_body">
     <inertial>
-      <mass value = "1.086" />
+      <mass value = "1.586" />
       <origin xyz="0 0 0.00907" rpy="0 0 0"/>
       <inertia
-          ixx="0.0777" ixy="0.00178" ixz="0.00000"
+          ixx="0.00777" ixy="0.000178" ixz="0"
           iyy="0.407" iyz="0"
           izz="0.412"/>
@@ -120,5 +120,5 @@
     </visual>
     <collision>
-      <origin rpy="0 0 3.14159265358979" xyz="0 0 0"/>
+      <origin rpy="0 0 0" xyz="0 0 0"/>
       <geometry>
         <box size="1.5 0.35 0.168" />
@@ -128,5 +128,5 @@
   <!-- spinal -->
   <xacro:extra_module name = "fc" parent = "main_body" visible = "0" >
-    <origin xyz="-0.613 0.0 0.0195" rpy="0 0 3.14159265358979"/>
+    <origin xyz="0.613 0.0 0.0195" rpy="0 0 3.14159265358979"/>
     <inertial>
       <mass value = "0.05" />

Commit message: [tilted_quadrotors] implemented SR-inverse based fully actuated control

File: robots/assemble_quadrotors/urdf/tilted/dual/robot1.urdf.xacro (robot description, xacro)
@@ -120,5 +120,5 @@
     </visual>
     <collision>
-      <origin rpy="0 0 3.14159265358979" xyz="0 0 0"/>
+      <origin rpy="0 0 0" xyz="0 0 0"/>
       <geometry>
         <box size="1.5 0.35 0.168" />

File: robots/assemble_quadrotors/urdf/tilted/dual/robot2.urdf.xacro (robot description, xacro)
@@ -128,5 +128,5 @@
   <!-- spinal -->
   <xacro:extra_module name = "fc" parent = "main_body" visible = "0" >
-    <origin xyz="0.613 0.0 0.0195" rpy="0 0 3.14159265358979"/>
+    <origin xyz="-0.613 0.0 0.0195" rpy="0 0 0"/>
     <inertial>
       <mass value = "0.05" />

Commit message: [model] updated model of quadrotors

File: robots/assemble_quadrotors/urdf/tilted/dual/robot1.urdf.xacro (robot description, xacro)
@@ -6,11 +6,11 @@
   <thrust_link name="thrust" />
   <!-- kinematics [m] -->
-  <xacro:property name="rotor_x_near" value="0.4991" />
-  <xacro:property name="rotor_y_near" value="0.1073" />
-  <xacro:property name="rotor_z_near" value="0.0351" />
-  <xacro:property name="rotor_x_far" value="0.7386" />
-  <xacro:property name="rotor_y_far" value="0.1077" />
-  <xacro:property name="rotor_z_far" value="0.0358" />
-  <xacro:property name="rotor_tilt" value="${pi/9}" />
+  <xacro:property name="rotor_x_near" value="0.468" />
+  <xacro:property name="rotor_y_near" value="0.131" />
+  <xacro:property name="rotor_z_near" value="0.0531" />
+  <xacro:property name="rotor_x_far" value="0.776" />
+  <xacro:property name="rotor_y_far" value="0.133" />
+  <xacro:property name="rotor_z_far" value="0.0509" />
+  <xacro:property name="rotor_tilt" value="${pi/4}" />
   <!-- dynamics -->
   <m_f_rate value="-0.006" /> <!-- drag torque rate, the true value should be -0.006 -->

File: robots/assemble_quadrotors/urdf/tilted/dual/robot2.urdf.xacro (robot description, xacro)
@@ -6,11 +6,11 @@
   <thrust_link name="thrust" />
   <!-- kinematics [m] -->
-  <xacro:property name="rotor_x_near" value="0.4991" />
-  <xacro:property name="rotor_y_near" value="0.1073" />
-  <xacro:property name="rotor_z_near" value="0.0351" />
-  <xacro:property name="rotor_x_far" value="0.7386" />
-  <xacro:property name="rotor_y_far" value="0.1077" />
-  <xacro:property name="rotor_z_far" value="0.0358" />
-  <xacro:property name="rotor_tilt" value="${pi/9}" />
+  <xacro:property name="rotor_x_near" value="0.468" />
+  <xacro:property name="rotor_y_near" value="0.131" />
+  <xacro:property name="rotor_z_near" value="0.0531" />
+  <xacro:property name="rotor_x_far" value="0.776" />
+  <xacro:property name="rotor_y_far" value="0.133" />
+  <xacro:property name="rotor_z_far" value="0.0509" />
+  <xacro:property name="rotor_tilt" value="${pi/4}" />
   <!-- dynamics -->
   <m_f_rate value="-0.006" /> <!-- drag torque rate, the true value should be -0.006 -->
