Commit message: [BEE][URDF] fix motor disposition and coordinate inertia

File: robots/gimbalrotor/robots/bee/gimbalrotor.urdf.xacro (robot description, xacro)
@@ -7,5 +7,5 @@
   <xacro:gimbalrotor_thrust_link self="1" rotor_direction="1"/>
   <xacro:gimbalrotor_thrust_link self="2" rotor_direction="-1"/>
-  <xacro:gimbalrotor_thrust_link self="3" rotor_direction="1"/>
-  <xacro:gimbalrotor_thrust_link self="4" rotor_direction="-1"/>
+  <xacro:gimbalrotor_thrust_link self="3" rotor_direction="-1"/>
+  <xacro:gimbalrotor_thrust_link self="4" rotor_direction="1"/>
 </robot>

File: robots/gimbalrotor/urdf/bee/gimbalrotor.urdf.xacro (robot description, xacro)
@@ -22,12 +22,11 @@
     ## link
     <link name="base_link">
-      <inertial>
-        <origin xyz="-0.00055912 -0.00191842 0.00251468" rpy="0 0 0"/>
-        <mass value="1.096"/>
-        <inertia
-            ixx="0.00372944293" ixy="0.00000575009" ixz="-0.00002212425"
-            iyy="0.00311904098" iyz="0.00010503988"
-            izz="0.00431356116"
-            />
+      <origin xyz="-0.00055912 -0.00191842 0.00239942" rpy="0 0 0"/>
+      <inertial>
+        <mass value="1.14109090632"/>
+        <inertia
+            ixx="0.00357218934" ixy="0.00000546201" ixz="-0.00002108293"
+            iyy="0.00299236824" iyz="0.00009954722"
+            izz="0.00409717232"/>
       </inertial>
       <visual>
@@ -58,5 +57,5 @@
       <child link="fc"/>
       <parent link="base_link"/>
-      <origin rpy="0 0 0" xyz="0 0 0.07"/>
+      <origin rpy="0 0 0" xyz="-0.0175 0 0.07"/>
       <axis xyz="0 0 1"/>
     </joint>
@@ -107,21 +106,21 @@
       <parent link="base_link"/>
       <child link="rotor_arm${child3}"/>
+      <origin rpy="0 0 ${3/2*pi}" xyz="0.0 -0.051 0.0"/>
+      <axis xyz="0 0 1"/>
+    </joint>
+    <link name="rotor_arm${child4}">
+      <inertial>
+        <origin xyz="0 0 0" rpy="0 0 0"/>
+        <mass value="0.00001"/>
+        <inertia
+            ixx="0.0000001" ixy="0.0" ixz="0.0"
+            iyy="0.0000001" iyz="0.0"
+            izz="0.0000001"/>
+      </inertial>
+    </link>
+    <joint name="base_arm_joint${child4}" type="fixed">
+      <parent link="base_link"/>
+      <child link="rotor_arm${child4}"/>
       <origin rpy="0 0 ${pi}" xyz="-0.051 0.0 0.0"/>
-      <axis xyz="0 0 1"/>
-    </joint>
-    <link name="rotor_arm${child4}">
-      <inertial>
-        <origin xyz="0 0 0" rpy="0 0 0"/>
-        <mass value="0.00001"/>
-        <inertia
-            ixx="0.0000001" ixy="0.0" ixz="0.0"
-            iyy="0.0000001" iyz="0.0"
-            izz="0.0000001"/>
-      </inertial>
-    </link>
-    <joint name="base_arm_joint${child4}" type="fixed">
-      <parent link="base_link"/>
-      <child link="rotor_arm${child4}"/>
-      <origin rpy="0 0 ${pi*3/2}" xyz="0.0 -0.051 0.0"/>
       <axis xyz="0 0 1"/>
     </joint>
