Commit message: [BEE] change propeller direction to downward

File: robots/gimbalrotor/urdf/bee/gimbalrotor.urdf.xacro (robot description, xacro)
@@ -23,13 +23,10 @@
     <link name="base_link">
       <inertial>
+        <origin xyz="-0.00055912 -0.00191842 0.00251468" rpy="0 0 0"/>
         <mass value="1.096"/>
-        <origin xyz="-0.00191842 0.00055912 0.00251468" rpy="0 0 0"/>
-        <inertia
-            ixx="0.00311483956"
-            ixy="-0.00000575009"
-            ixz="0.00010503988"
-            iyy="0.00372524151"
-            iyz="0.00002212425"
-            izz="0.00430515832"
+        <inertia
+            ixx="0.00372944293" ixy="0.00000575009" ixz="-0.00002212425"
+            iyy="0.00311904098" iyz="0.00010503988"
+            izz="0.00431356116"
             />
       </inertial>
@@ -135,17 +132,14 @@
     #### rotor parent link (virtual) ####
     <link name="gimbal_link${self}">
-    <inertial>
-      <mass value="0.04944"/>
-      <origin xyz="0.02631527 0.03530709 -0.07078771" rpy="0 0 0"/>
-      <inertia
-        ixx="0.00001018740"
-        ixy="-0.00000000588"
-        ixz="-0.00000168229"
-        iyy="0.00001158109"
-        iyz="-0.00000000185"
-        izz="0.00001165546"
-      />
-    </inertial>
-    <collision>
+      <inertial>
+        <origin xyz="0.01483947 0.00001426 -0.02606996" rpy="0 0 0"/>
+        <mass value="0.04944"/>
+        <inertia
+            ixx="0.00001165546" ixy="-0.00000000185" ixz="-0.00000168229"
+            iyy="0.00001158109" iyz="-0.00000000588"
+            izz="0.00001018740"
+            />
+      </inertial>
+      <collision>
         <origin xyz="0.0 0 0" rpy="0 0 0"/>
         <geometry>
@@ -156,5 +150,5 @@
         <origin xyz="0 0 0" rpy="0 0 0"/>
         <geometry>
-          <mesh filename="package://gimbalrotor/urdf/bee/mesh/rotor_module.STL"/>
+          <mesh filename="package://gimbalrotor/urdf/bee/mesh/rotor_module_downward.STL"/>
         </geometry>
       </visual>
@@ -216,5 +210,5 @@
       <parent link="rotor_parent${self}"/>
       <child link="thrust${self}"/>
-      <origin rpy="0 0 0" xyz="0 0 0"/>
+      <origin rpy="0 0 0" xyz="0 0 -0.04"/>
       <axis xyz="0 0 ${rotor_direction}"/>
     </joint>

Commit message: [BEE][URDF] change model to include Lidar

File: robots/gimbalrotor/urdf/bee/gimbalrotor.urdf.xacro (robot description, xacro)
@@ -74,5 +74,5 @@
       <parent link="base_link"/>
       <child link="rotor_arm${child1}"/>
-      <origin rpy="0 0 0" xyz="0.051 0.0 0.0"/>
+      <origin rpy="0 0 ${pi/4}" xyz="0.036 0.036 0.0"/>
       <axis xyz="0 0 1"/>
     </joint>
@@ -90,5 +90,5 @@
       <parent link="base_link"/>
       <child link="rotor_arm${child2}"/>
-      <origin rpy="0 0 ${pi/2}" xyz="0.0 0.051 0.0"/>
+      <origin rpy="0 0 ${3*pi/4}" xyz="-0.036 0.036 0.0"/>
       <axis xyz="0 0 1"/>
     </joint>
@@ -106,5 +106,5 @@
       <parent link="base_link"/>
       <child link="rotor_arm${child3}"/>
-      <origin rpy="0 0 ${3/2*pi}" xyz="0.0 -0.051 0.0"/>
+      <origin rpy="0 0 -${1/4*pi}" xyz="0.036 -0.036 0.0"/>
       <axis xyz="0 0 1"/>
     </joint>
@@ -122,5 +122,5 @@
       <parent link="base_link"/>
       <child link="rotor_arm${child4}"/>
-      <origin rpy="0 0 ${pi}" xyz="-0.051 0.0 0.0"/>
+      <origin rpy="0 0 -${3/4*pi}" xyz="-0.036 -0.036 0.0"/>
       <axis xyz="0 0 1"/>
     </joint>

Commit message: [Bee][URDF] fix inertia infomation

File: robots/gimbalrotor/urdf/bee/gimbalrotor.urdf.xacro (robot description, xacro)
@@ -22,11 +22,11 @@
     ## link
     <link name="base_link">
-      <origin xyz="-0.00055912 -0.00191842 0.00239942" rpy="0 0 0"/>
-      <inertial>
-        <mass value="1.14109090632"/>
-        <inertia
-            ixx="0.00357218934" ixy="0.00000546201" ixz="-0.00002108293"
-            iyy="0.00299236824" iyz="0.00009954722"
-            izz="0.00409717232"/>
+      <inertial>
+        <origin xyz="-0.00078520 0.00096010 0.01594366" rpy="0 0 0" />
+        <mass value="1.40419" />
+        <inertia
+            ixx="0.00607504" ixy="0.00014664"  ixz="0.00004521"
+            iyy="0.00609952" iyz="-0.00005926"
+            izz="0.00468030" />
       </inertial>
       <visual>

Commit message: [BEE][URDF] change position of fc

File: robots/gimbalrotor/urdf/bee/gimbalrotor.urdf.xacro (robot description, xacro)
@@ -57,5 +57,5 @@
       <child link="fc"/>
       <parent link="base_link"/>
-      <origin rpy="0 0 0" xyz="-0.0175 0 0.07"/>
+      <origin rpy="0 0 0" xyz="-0.0175 0 0.0375"/>
       <axis xyz="0 0 1"/>
     </joint>
