Commit message: add zedXmini mesh

File: robots/gimbalrotor/urdf/ynltilt/zed_macro.urdf.xacro (robot description, xacro)
@@ -86,5 +86,5 @@
         <origin xyz="${screw_offset_x} 0 ${screw_offset_z}" rpy="0 0 0"/>
         <geometry>
-          <mesh filename="package://zed_interfaces/meshes/${model}.stl" />
+          <mesh filename="meshes/${model}.stl" />
         </geometry>
         <material name="${model}_mat" />
@@ -92,5 +92,5 @@
       <collision>
         <geometry>
-          <mesh filename="package://zed_interfaces/meshes/${model}.stl" />
+          <mesh filename="meshes/${model}.stl" />
         </geometry>
       </collision>
