Commit message: Commented the Prunning Tools

File: robots/gimbalrotor/urdf/ynltilt/gimbalrotor.urdf.xacro (robot description, xacro)
@@ -22,5 +22,6 @@
     ## link
     <link name="base_link">
-      <!-- <inertial>
+      <!--Without Prunning Tools-->
+      <inertial>
         <origin xyz="0.00009021 -0.00005299 0.04639014" rpy="0 0 0"/>
         <mass value="1.16544411"/>
@@ -28,6 +29,7 @@
             ixx="0.01251517" iyy="0.01254829" izz="0.01920936"
             ixy="-0.00000046" ixz="-0.00000278" iyz="-0.00001104"/>
-      </inertial> -->
-      <inertial>
+      </inertial>
+      <!--With Prunning Tools-->
+      <!-- <inertial>
         <origin xyz="0.05984 0.00138 0.03247" rpy="0 0 0"/>
         <mass value="1.43147"/>
@@ -36,5 +38,5 @@
             iyx="-0.00059865083" iyy="0.03783180404" iyz="-0.00018635030"
             izx="-0.00538129912" izy="-0.00018635030" izz="0.04319444852"/>
-      </inertial>
+      </inertial> -->
       <visual>
         <origin xyz="0 0 -0.0" rpy="0 0 0"/>

Commit message: update Inertial matrix in URDF: with zedXmini

File: robots/gimbalrotor/urdf/ynltilt/gimbalrotor.urdf.xacro (robot description, xacro)
@@ -22,6 +22,17 @@
     ## link
     <link name="base_link">
+      <!-- Inertial must be calculate in COG -->
+      <!--with Pruning-Tool and ZED-X-mini-->
+      <inertial>
+        <origin xyz="0.4193 0 0.4581" rpy="0 0 0"/> <!-- unit=meter -->
+        <mass value="2.15088"/> <!-- Unit=kg -->
+        <!-- Unit=kg*m*m and SolidWorks is in g*mm*mm, so *10^-9 to convert the unit. -->
+        <inertia
+            ixx="0.02834257041" ixy="0.00079044376" ixz="-0.00444925108"
+            iyx="0.00079044376" iyy="0.05504841972" iyz="-0.00032810096"
+            izx="-0.00444925108" izy="-0.00032810096" izz="0.07516900973"/>
+      </inertial>
       <!--Without Prunning Tools-->
-      <inertial>
+      <!-- <inertial>
         <origin xyz="0.00009021 -0.00005299 0.04639014" rpy="0 0 0"/>
         <mass value="1.16544411"/>
@@ -29,5 +40,5 @@
             ixx="0.01251517" iyy="0.01254829" izz="0.01920936"
             ixy="-0.00000046" ixz="-0.00000278" iyz="-0.00001104"/>
-      </inertial>
+      </inertial> -->
       <!--With Prunning Tools-->
       <!-- <inertial>

Commit message: update URDF for zedXmini: note that 'catkin build' was run, so other members may have to re-build before they run roslaunch

File: robots/gimbalrotor/urdf/ynltilt/gimbalrotor.urdf.xacro (robot description, xacro)
@@ -2,4 +2,6 @@
 <robot
     xmlns:xacro="http://www.ros.org/wiki/xacro" name="gimbalrotor_link" >
+  <!-- Include ZED camera macro -->
+  <xacro:include filename="zed_macro.urdf.xacro" />
   <xacro:macro name="gimbalrotor_center_link" params="child1 child2 child3 child4">
     ## dummy
@@ -146,4 +148,9 @@
     </joint>
     <xacro:friction self="base_link"/>
+    <!-- ZED X MINI Camera Integration -->
+    <xacro:zed_camera name="zedxm" model="zedxm" parent="base_link">
+      <!-- ドローン原点からZED X MINIのねじ穴までの相対座標-->
+      <origin xyz="0.08318 0.0 0.027" rpy="0 0 0" />
+    </xacro:zed_camera>
   </xacro:macro>
   <xacro:macro name="gimbalrotor_thrust_link" params="self rotor_direction">

Commit message: urdf update teamp

File: robots/gimbalrotor/urdf/ynltilt/gimbalrotor.urdf.xacro (robot description, xacro)
@@ -24,17 +24,17 @@
     ## link
     <link name="base_link">
-      <!-- Inertial must be calculate in COG -->
+      <!-- Inertial must be calculate in COG and multiple 10^9 against SolidWorks output -->
       <!--with Pruning-Tool and ZED-X-mini-->
-      <inertial>
-        <origin xyz="0.4193 0 0.4581" rpy="0 0 0"/> <!-- unit=meter -->
-        <mass value="2.15088"/> <!-- Unit=kg -->
-        <!-- Unit=kg*m*m and SolidWorks is in g*mm*mm, so *10^-9 to convert the unit. -->
+	<!-- <inertial>
+        <origin xyz="0.4193 0 0.4581" rpy="0 0 0"/>
+        <mass value="2.15088"/>
         <inertia
             ixx="0.02834257041" ixy="0.00079044376" ixz="-0.00444925108"
             iyx="0.00079044376" iyy="0.05504841972" iyz="-0.00032810096"
             izx="-0.00444925108" izy="-0.00032810096" izz="0.07516900973"/>
-      </inertial>
+	</inertial>
+	-->
       <!--Without Prunning Tools-->
-      <!-- <inertial>
+      <!--<inertial>
         <origin xyz="0.00009021 -0.00005299 0.04639014" rpy="0 0 0"/>
         <mass value="1.16544411"/>
@@ -42,7 +42,8 @@
             ixx="0.01251517" iyy="0.01254829" izz="0.01920936"
             ixy="-0.00000046" ixz="-0.00000278" iyz="-0.00001104"/>
-      </inertial> -->
+	      </inertial>
+      -->
       <!--With Prunning Tools-->
-      <!-- <inertial>
+      <inertial>
         <origin xyz="0.05984 0.00138 0.03247" rpy="0 0 0"/>
         <mass value="1.43147"/>
@@ -51,5 +52,5 @@
             iyx="-0.00059865083" iyy="0.03783180404" iyz="-0.00018635030"
             izx="-0.00538129912" izy="-0.00018635030" izz="0.04319444852"/>
-      </inertial> -->
+	</inertial>
       <visual>
         <origin xyz="0 0 -0.0" rpy="0 0 0"/>

Commit message: update urdf for sector gear and zedXmini

File: robots/gimbalrotor/urdf/ynltilt/gimbalrotor.urdf.xacro (robot description, xacro)
@@ -25,14 +25,13 @@
     <link name="base_link">
       <!-- Inertial must be calculate in COG and multiple 10^9 against SolidWorks output -->
-      <!--with Pruning-Tool and ZED-X-mini-->
-	<!-- <inertial>
-        <origin xyz="0.4193 0 0.4581" rpy="0 0 0"/>
-        <mass value="2.15088"/>
-        <inertia
-            ixx="0.02834257041" ixy="0.00079044376" ixz="-0.00444925108"
-            iyx="0.00079044376" iyy="0.05504841972" iyz="-0.00032810096"
-            izx="-0.00444925108" izy="-0.00032810096" izz="0.07516900973"/>
+      <!--with Pruning-Tool-Sector and ZED-X-mini-->
+	<inertial>
+        <origin xyz="0.6353 -0.0527 0.4362" rpy="0 0 0"/>
+        <mass value="2.32375"/>
+        <inertia
+            ixx="0.03008400484" ixy="-0.00297777401" ixz="-0.00664821011"
+            iyx="-0.00297777401" iyy="0.06882060466" iyz="0.00047002139"
+            izx="-0.00664821011" izy="0.00047002139" izz="0.08922548478"/>
 	</inertial>
-	-->
       <!--Without Prunning Tools-->
       <!--<inertial>

Commit message: refactor urdf

File: robots/gimbalrotor/urdf/ynltilt/gimbalrotor.urdf.xacro (robot description, xacro)
@@ -44,5 +44,5 @@
       -->
       <!--With Prunning Tools-->
-      <inertial>
+ <!--     <inertial>
         <origin xyz="0.05984 0.00138 0.03247" rpy="0 0 0"/>
         <mass value="1.43147"/>
@@ -52,4 +52,5 @@
             izx="-0.00538129912" izy="-0.00018635030" izz="0.04319444852"/>
 	</inertial>
+-->
       <visual>
         <origin xyz="0 0 -0.0" rpy="0 0 0"/>

Commit message: fix COG

File: robots/gimbalrotor/urdf/ynltilt/gimbalrotor.urdf.xacro (robot description, xacro)
@@ -27,5 +27,5 @@
       <!--with Pruning-Tool-Sector and ZED-X-mini-->
 	<inertial>
-        <origin xyz="0.6353 -0.0527 0.4362" rpy="0 0 0"/>
+        <origin xyz="0.06353 -0.00527 0.04362" rpy="0 0 0"/>
         <mass value="2.32375"/>
         <inertia
@@ -44,5 +44,5 @@
       -->
       <!--With Prunning Tools-->
- <!--     <inertial>
+      <!-- <inertial>
         <origin xyz="0.05984 0.00138 0.03247" rpy="0 0 0"/>
         <mass value="1.43147"/>
@@ -52,5 +52,5 @@
             izx="-0.00538129912" izy="-0.00018635030" izz="0.04319444852"/>
 	</inertial>
--->
+      -->
       <visual>
         <origin xyz="0 0 -0.0" rpy="0 0 0"/>

Commit message: update LiDAR position

File: robots/gimbalrotor/urdf/ynltilt/gimbalrotor.urdf.xacro (robot description, xacro)
@@ -270,5 +270,5 @@
   </xacro:macro>
   <xacro:extra_module name = "lidar_imu" parent = "base_link" visible = "0" > <!-- should be IMU frame -->
-    <origin xyz="${0.0} ${0.0} ${0.145}" rpy="0 0 ${-pi/2.0}"/> <!-- TODO: the true pos -->
+    <origin xyz="${0.0} ${0.0} ${0.16082}" rpy="0 0 ${-pi/2.0}"/> <!-- TODO: the true pos -->
     <inertial>
       <mass value = "00" />

Commit message: add zedXmini in URDF properly

File: robots/gimbalrotor/urdf/ynltilt/gimbalrotor.urdf.xacro (robot description, xacro)
@@ -25,6 +25,15 @@
     <link name="base_link">
       <!-- Inertial must be calculate in COG and multiple 10^9 against SolidWorks output -->
-      <!--with Pruning-Tool-Sector and ZED-X-mini-->
-	<inertial>
+    <!--With Pruning-Tool-Sector and zedXmini ON THE PLATE-->
+      <inertial>
+            <origin xyz="0.06310 -0.00517 0.05062" rpy="0 0 0"/>
+            <mass value="2.33579"/>
+            <inertia
+                ixx="0.03008400484" ixy="-0.00297777401" ixz="-0.00664821011"
+                iyx="-0.00297777401" iyy="0.06882060466" iyz="0.00047002139"
+                izx="-0.00664821011" izy="0.00047002139" izz="0.08922548478"/>
+      </inertial>
+      <!--with Pruning-Tool-Sector and zedXmini BETWEEN PLATES-->
+<!--      <inertial>
         <origin xyz="0.06353 -0.00527 0.04362" rpy="0 0 0"/>
         <mass value="2.32375"/>
@@ -33,5 +42,6 @@
             iyx="-0.00297777401" iyy="0.06882060466" iyz="0.00047002139"
             izx="-0.00664821011" izy="0.00047002139" izz="0.08922548478"/>
-	</inertial>
+	    </inertial>
+-->
       <!--Without Prunning Tools-->
       <!--<inertial>
@@ -151,6 +161,6 @@
     <!-- ZED X MINI Camera Integration -->
     <xacro:zed_camera name="zedxm" model="zedxm" parent="base_link">
-      <!-- ドローン原点からZED X MINIのねじ穴までの相対座標-->
-      <origin xyz="0.08318 0.0 0.027" rpy="0 0 0" />
+      <!-- ドローン原点からzedXminiのねじ穴までの相対座標（ZED on TOP plate）-->
+      <origin xyz="0.08653 0.0 0.09595" rpy="0 0 0" />
     </xacro:zed_camera>
   </xacro:macro>

Commit message: fix inertia in URDF

File: robots/gimbalrotor/urdf/ynltilt/gimbalrotor.urdf.xacro (robot description, xacro)
@@ -289,3 +289,32 @@
     </inertial>
   </xacro:extra_module>
+    <!-- Arm (Scissors) rotation center -->
+  <xacro:extra_module name="scissor_center" parent="base_link" visible="1">
+    <origin xyz="0.42126 -0.0154 -0.0003" rpy="0 0 0"/>
+    <inertial>
+      <mass value="0.00001"/>
+      <origin xyz="0 0 0" rpy="0 0 0"/>
+      <inertia
+          ixx="0.000001" ixy="0.0" ixz="0.0"
+          iyy="0.000001" iyz="0.0" izz="0.000001"/>
+    </inertial>
+  </xacro:extra_module>
+  <link name="arm_link_1">
+    <inertial>
+      <mass value="0.001"/>
+      <origin xyz="0 0 0" rpy="0 0 0"/>
+      <inertia ixx="1e-6" ixy="0" ixz="0" iyy="1e-6" iyz="0" izz="1e-6"/>
+    </inertial>
+    <visual>
+      <origin xyz="0 0 0" rpy="0 0 0"/>
+      <geometry>
+        <box size="0.02 0.02 0.02"/>
+      </geometry>
+    </visual>
+  </link>
+  <joint name="scissor_joint" type="fixed">
+    <parent link="scissor_center"/>
+    <child link="arm_link_1"/>
+    <origin xyz="0 0 0" rpy="0 0 0"/>
+  </joint>
 </robot>
