Commit message: refactor: update gimbal controller gains/urdf and remove unused files

File: robots/gimbalrotor/urdf/ynltilt/gimbalrotor.urdf.xacro (robot description, xacro)
@@ -2,6 +2,4 @@
 <robot
     xmlns:xacro="http://www.ros.org/wiki/xacro" name="gimbalrotor_link" >
-  <!-- Include ZED camera macro -->
-  <xacro:include filename="zed_macro.urdf.xacro" />
   <xacro:macro name="gimbalrotor_center_link" params="child1 child2 child3 child4">
     ## dummy
@@ -24,43 +22,11 @@
     ## link
     <link name="base_link">
-      <!-- Inertial must be calculate in COG and multiple 10^9 against SolidWorks output -->
-    <!--With Pruning-Tool-Sector and zedXmini ON THE PLATE-->
-      <inertial>
-            <origin xyz="0.06310 -0.00517 0.05062" rpy="0 0 0"/>
-            <mass value="2.33579"/>
-            <inertia
-                ixx="0.03008400484" ixy="-0.00297777401" ixz="-0.00664821011"
-                iyx="-0.00297777401" iyy="0.06882060466" iyz="0.00047002139"
-                izx="-0.00664821011" izy="0.00047002139" izz="0.08922548478"/>
-      </inertial>
-      <!--with Pruning-Tool-Sector and zedXmini BETWEEN PLATES-->
-<!--      <inertial>
-        <origin xyz="0.06353 -0.00527 0.04362" rpy="0 0 0"/>
-        <mass value="2.32375"/>
-        <inertia
-            ixx="0.03008400484" ixy="-0.00297777401" ixz="-0.00664821011"
-            iyx="-0.00297777401" iyy="0.06882060466" iyz="0.00047002139"
-            izx="-0.00664821011" izy="0.00047002139" izz="0.08922548478"/>
-	    </inertial>
--->
-      <!--Without Prunning Tools-->
-      <!--<inertial>
-        <origin xyz="0.00009021 -0.00005299 0.04639014" rpy="0 0 0"/>
-        <mass value="1.16544411"/>
-        <inertia
-            ixx="0.01251517" iyy="0.01254829" izz="0.01920936"
-            ixy="-0.00000046" ixz="-0.00000278" iyz="-0.00001104"/>
+      <inertial>
+        <origin xyz="0.00007563 0.00006801 0.04457233" rpy="0 0 0"/>
+        <mass value="1.60833857"/>
+        <inertia
+            ixx="0.01841510" iyy="0.01843894" izz="0.02261725"
+            ixy="-0.00000048" ixz="0.00000375" iyz="0.00000647"/>
 	      </inertial>
-      -->
-      <!--With Prunning Tools-->
-      <!-- <inertial>
-        <origin xyz="0.05984 0.00138 0.03247" rpy="0 0 0"/>
-        <mass value="1.43147"/>
-        <inertia
-            ixx="0.01393149076" ixy="0.00059865083" ixz="-0.00538129912"
-            iyx="-0.00059865083" iyy="0.03783180404" iyz="-0.00018635030"
-            izx="-0.00538129912" izy="-0.00018635030" izz="0.04319444852"/>
-	</inertial>
-      -->
       <visual>
         <origin xyz="0 0 -0.0" rpy="0 0 0"/>
@@ -159,9 +125,4 @@
     </joint>
     <xacro:friction self="base_link"/>
-    <!-- ZED X MINI Camera Integration -->
-    <xacro:zed_camera name="zedxm" model="zedxm" parent="base_link">
-      <!-- ドローン原点からzedXminiのねじ穴までの相対座標（ZED on TOP plate）-->
-      <origin xyz="0.08653 0.0 0.09595" rpy="0 0 0" />
-    </xacro:zed_camera>
   </xacro:macro>
   <xacro:macro name="gimbalrotor_thrust_link" params="self rotor_direction">
@@ -170,10 +131,10 @@
     <link name="gimbal_link${self}">
       <inertial>
-        <origin xyz="0.0412 0.00 0.0184" rpy="0 0 0"/>
-        <mass value="0.14"/>
-        <inertia
-            ixx="0.00003614" ixy="0.0000"     ixz="0.00000471"
-                             iyy="0.00004251" iyz="0.00000"
-                                              izz="0.00002946"
+        <origin xyz="0.0471 0.00 0.016269" rpy="0 0 0"/>
+        <mass value="0.1570"/>
+        <inertia
+            ixx="0.00009933" ixy="0.0000"     ixz="0.00011468"
+                             iyy="0.00052148" iyz="0.00000"
+                                              izz="0.00047583"
         />
       </inertial>
@@ -239,5 +200,5 @@
       <parent link="gimbal_link${self}"/>
       <child link="rotor_parent${self}"/>
-      <origin rpy="0 0 0" xyz="0.0205 0.00 0.03515"/>
+      <origin rpy="0 0 0" xyz="0.045 0.0 0.00175"/> <!-- servo horn -> motor base on the cantilever -->
       <axis xyz="0 0 ${rotor_direction}"/>
     </joint>
@@ -247,5 +208,5 @@
       <parent link="rotor_parent${self}"/>
       <child link="thrust${self}"/>
-      <origin rpy="0 0 0" xyz="0 0 0"/>
+      <origin rpy="0 0 0" xyz="0.0 0.0 0.020"/> <!-- motor base -> propeller disc -->
       <axis xyz="0 0 ${rotor_direction}"/>
     </joint>
@@ -279,6 +240,6 @@
     </link>
   </xacro:macro>
-  <xacro:extra_module name = "lidar_imu" parent = "base_link" visible = "0" > <!-- should be IMU frame -->
-    <origin xyz="${0.0} ${0.0} ${0.16082}" rpy="0 0 ${-pi/2.0}"/> <!-- TODO: the true pos -->
+  <xacro:extra_module name = "lidar_imu" parent = "base_link" visible = "0" >
+    <origin xyz="${0.0} ${0.0} ${0.15562}" rpy="0 0 ${-pi/2.0}"/>
     <inertial>
       <mass value = "00" />
@@ -289,32 +250,3 @@
     </inertial>
   </xacro:extra_module>
-    <!-- Arm (Scissors) rotation center -->
-  <xacro:extra_module name="scissor_center" parent="base_link" visible="1">
-    <origin xyz="0.42126 -0.0154 -0.0003" rpy="0 0 0"/>
-    <inertial>
-      <mass value="0.00001"/>
-      <origin xyz="0 0 0" rpy="0 0 0"/>
-      <inertia
-          ixx="0.000001" ixy="0.0" ixz="0.0"
-          iyy="0.000001" iyz="0.0" izz="0.000001"/>
-    </inertial>
-  </xacro:extra_module>
-  <link name="arm_link_1">
-    <inertial>
-      <mass value="0.001"/>
-      <origin xyz="0 0 0" rpy="0 0 0"/>
-      <inertia ixx="1e-6" ixy="0" ixz="0" iyy="1e-6" iyz="0" izz="1e-6"/>
-    </inertial>
-    <visual>
-      <origin xyz="0 0 0" rpy="0 0 0"/>
-      <geometry>
-        <box size="0.02 0.02 0.02"/>
-      </geometry>
-    </visual>
-  </link>
-  <joint name="scissor_joint" type="fixed">
-    <parent link="scissor_center"/>
-    <child link="arm_link_1"/>
-    <origin xyz="0 0 0" rpy="0 0 0"/>
-  </joint>
 </robot>

Commit message: fix: thrust location of ynltilt gimbalrotor

File: robots/gimbalrotor/urdf/ynltilt/gimbalrotor.urdf.xacro (robot description, xacro)
@@ -208,5 +208,5 @@
       <parent link="rotor_parent${self}"/>
       <child link="thrust${self}"/>
-      <origin rpy="0 0 0" xyz="0.0 0.0 0.020"/> <!-- motor base -> propeller disc -->
+      <origin rpy="0 0 0" xyz="0.0 0.0 0.0425"/> <!-- motor base -> propeller disc -->
       <axis xyz="0 0 ${rotor_direction}"/>
     </joint>

Commit message: fix(ynltilt): make LiDAR IMU location more accurate

File: robots/gimbalrotor/urdf/ynltilt/gimbalrotor.urdf.xacro (robot description, xacro)
@@ -240,5 +240,5 @@
     </link>
   </xacro:macro>
-  <xacro:extra_module name = "lidar_imu" parent = "base_link" visible = "0" >
+  <xacro:extra_module name = "lidar_optical_center" parent = "base_link" visible = "0" >
     <origin xyz="${0.0} ${0.0} ${0.15562}" rpy="0 0 ${-pi/2.0}"/>
     <inertial>
@@ -250,3 +250,13 @@
     </inertial>
   </xacro:extra_module>
+  <xacro:extra_module name = "lidar_imu" parent = "lidar_optical_center" visible = "0" >
+    <origin xyz="${0.011} ${0.02329} ${-0.04412}" rpy="0 0 0"/>
+    <inertial>
+      <mass value = "00" />
+      <origin xyz="0 0 0" rpy="0 0 0"/>
+      <inertia
+          ixx="0.0" ixy="0.0" ixz="0.0"
+          iyy="0.0" iyz="0.0" izz="0.0"/>
+    </inertial>
+  </xacro:extra_module>
 </robot>

Commit message: fix(ynltilt): add small mass and inertia to LiDAR links

File: robots/gimbalrotor/urdf/ynltilt/gimbalrotor.urdf.xacro (robot description, xacro)
@@ -32,5 +32,5 @@
         <origin xyz="0 0 -0.0" rpy="0 0 0"/>
         <geometry>
-          <mesh filename="package://gimbalrotor/urdf/ynltilt/mesh/experiment_mode_noprop.STL"/>
+          <mesh filename="package://gimbalrotor/urdf/ynltilt/mesh/experiment_mode_noprop.stl"/>
         </geometry>
       </visual>
@@ -148,5 +148,5 @@
         <origin xyz="0 0 0" rpy="0 0 0"/>
         <geometry>
-          <mesh filename="package://gimbalrotor/urdf/ynltilt/mesh/prop_module_5in.STL"/>
+          <mesh filename="package://gimbalrotor/urdf/ynltilt/mesh/prop_module_5in.stl"/>
         </geometry>
       </visual>
@@ -243,9 +243,9 @@
     <origin xyz="${0.0} ${0.0} ${0.15562}" rpy="0 0 ${-pi/2.0}"/>
     <inertial>
-      <mass value = "00" />
+      <mass value = "0.00001" />
       <origin xyz="0 0 0" rpy="0 0 0"/>
       <inertia
-          ixx="0.0" ixy="0.0" ixz="0.0"
-          iyy="0.0" iyz="0.0" izz="0.0"/>
+          ixx="0.000001" ixy="0.0" ixz="0.0"
+          iyy="0.000001" iyz="0.0" izz="0.000001"/>
     </inertial>
   </xacro:extra_module>
@@ -253,9 +253,9 @@
     <origin xyz="${0.011} ${0.02329} ${-0.04412}" rpy="0 0 0"/>
     <inertial>
-      <mass value = "00" />
+      <mass value = "0.00001" />
       <origin xyz="0 0 0" rpy="0 0 0"/>
       <inertia
-          ixx="0.0" ixy="0.0" ixz="0.0"
-          iyy="0.0" iyz="0.0" izz="0.0"/>
+          ixx="0.000001" ixy="0.0" ixz="0.0"
+          iyy="0.000001" iyz="0.0" izz="0.000001"/>
     </inertial>
   </xacro:extra_module>

Commit message: feat(flex): use actual models and mount points

File: robots/gimbalrotor/urdf/ynltilt/gimbalrotor.urdf.xacro (robot description, xacro)
@@ -2,5 +2,6 @@
 <robot
     xmlns:xacro="http://www.ros.org/wiki/xacro" name="gimbalrotor_link" >
-  <xacro:macro name="gimbalrotor_center_link" params="child1 child2 child3 child4">
+  <xacro:include filename="$(find gimbalrotor)/urdf/ynltilt/macros.urdf.xacro" />
+  <xacro:macro name="gimbalrotor_center_link" params="child1 child2 child3 child4 mesh:=baseline_2026ver_noprop.stl">
     ## dummy
     <link name="root">
@@ -32,5 +33,5 @@
         <origin xyz="0 0 -0.0" rpy="0 0 0"/>
         <geometry>
-          <mesh filename="package://gimbalrotor/urdf/ynltilt/mesh/experiment_mode_noprop.stl"/>
+          <mesh filename="package://gimbalrotor/urdf/ynltilt/mesh/${mesh}"/>
         </geometry>
       </visual>
@@ -148,5 +149,5 @@
         <origin xyz="0 0 0" rpy="0 0 0"/>
         <geometry>
-          <mesh filename="package://gimbalrotor/urdf/ynltilt/mesh/prop_module_5in.stl"/>
+          <mesh filename="package://gimbalrotor/urdf/ynltilt/mesh/prop_module_9in_v2.stl"/>
         </geometry>
       </visual>
@@ -225,22 +226,4 @@
       </actuator>
     </transmission>
-  </xacro:macro>
-  <xacro:macro name="extra_module" params="name parent *origin *inertial visible:=0 model_url:=1 scale:=1">
-    <joint name="${parent}2${name}" type="fixed">
-      <parent link="${parent}"/>
-      <child link="${name}"/>
-      <xacro:insert_block name="origin" />
-    </joint>
-    <link name="${name}">
-      <xacro:insert_block name="inertial" />
-      <xacro:if value="${visible == 1}">
-        <visual>
-          <origin rpy="0 0 0" xyz="0 0 0"/>
-          <geometry>
-            <mesh filename="${model_url}" scale= "${scale} ${scale} ${scale}"/>
-          </geometry>
-        </visual>
-      </xacro:if>
-    </link>
   </xacro:macro>
   <xacro:extra_module name = "lidar_optical_center" parent = "base_link" visible = "0" >
