Commit message: feat: integrate mujoco support and enhance ground truth functionality for gimbalrotor

File: robots/gimbalrotor/urdf/quad/gimbalrotor.urdf.xacro (robot description, xacro)
@@ -32,5 +32,5 @@
         <origin xyz="0 0 -0.0165" rpy="0 0 0"/>
         <geometry>
-          <mesh filename="package://gimbalrotor/urdf/quad/mesh/base_link.STL"/>
+          <mesh filename="package://gimbalrotor/urdf/quad/mesh/base_link.stl"/>
         </geometry>
       </visual>
@@ -72,5 +72,5 @@
         <origin xyz="0 0 0" rpy="0 0 0"/>
         <geometry>
-          <mesh filename="package://gimbalrotor/urdf/quad/mesh/rotor_arm.STL"/>
+          <mesh filename="package://gimbalrotor/urdf/quad/mesh/rotor_arm.stl"/>
         </geometry>
       </visual>
@@ -100,5 +100,5 @@
         <origin xyz="0 0 0" rpy="0 0 0"/>
         <geometry>
-          <mesh filename="package://gimbalrotor/urdf/quad/mesh/rotor_arm.STL"/>
+          <mesh filename="package://gimbalrotor/urdf/quad/mesh/rotor_arm.stl"/>
         </geometry>
       </visual>
@@ -128,5 +128,5 @@
         <origin xyz="0 0 0" rpy="0 0 0"/>
         <geometry>
-          <mesh filename="package://gimbalrotor/urdf/quad/mesh/rotor_arm.STL"/>
+          <mesh filename="package://gimbalrotor/urdf/quad/mesh/rotor_arm.stl"/>
         </geometry>
       </visual>
@@ -156,5 +156,5 @@
         <origin xyz="0 0 0" rpy="0 0 0"/>
         <geometry>
-          <mesh filename="package://gimbalrotor/urdf/quad/mesh/rotor_arm.STL"/>
+          <mesh filename="package://gimbalrotor/urdf/quad/mesh/rotor_arm.stl"/>
         </geometry>
       </visual>
@@ -194,5 +194,5 @@
         <origin xyz="0 0 0" rpy="0 0 0"/>
         <geometry>
-          <mesh filename="package://gimbalrotor/urdf/quad/mesh/rotor_module.STL"/>
+          <mesh filename="package://gimbalrotor/urdf/quad/mesh/rotor_module.stl"/>
         </geometry>
       </visual>

File: robots/gimbalrotor/urdf/ynltilt/gimbalrotor.urdf.xacro (robot description, xacro)
@@ -32,5 +32,5 @@
         <origin xyz="0 0 -0.0" rpy="0 0 0"/>
         <geometry>
-          <mesh filename="package://gimbalrotor/urdf/ynltilt/mesh/experiment_mode_noprop.STL"/>
+          <mesh filename="package://gimbalrotor/urdf/ynltilt/mesh/experiment_mode_noprop.stl"/>
         </geometry>
       </visual>
@@ -148,5 +148,5 @@
         <origin xyz="0 0 0" rpy="0 0 0"/>
         <geometry>
-          <mesh filename="package://gimbalrotor/urdf/ynltilt/mesh/prop_module_5in.STL"/>
+          <mesh filename="package://gimbalrotor/urdf/ynltilt/mesh/prop_module_5in.stl"/>
         </geometry>
       </visual>

Commit message: feat(mujoco): add prefix-aware shared MuJoCo 3 simulation for mini_quadrotor and gimbalrotor

File: robots/gimbalrotor/urdf/quad/gimbalrotor.urdf.xacro (robot description, xacro)
@@ -32,5 +32,5 @@
         <origin xyz="0 0 -0.0165" rpy="0 0 0"/>
         <geometry>
-          <mesh filename="package://gimbalrotor/urdf/quad/mesh/base_link.STL"/>
+          <mesh filename="package://gimbalrotor/urdf/quad/mesh/base_link.stl"/>
         </geometry>
       </visual>
@@ -72,5 +72,5 @@
         <origin xyz="0 0 0" rpy="0 0 0"/>
         <geometry>
-          <mesh filename="package://gimbalrotor/urdf/quad/mesh/rotor_arm.STL"/>
+          <mesh filename="package://gimbalrotor/urdf/quad/mesh/rotor_arm.stl"/>
         </geometry>
       </visual>
@@ -100,5 +100,5 @@
         <origin xyz="0 0 0" rpy="0 0 0"/>
         <geometry>
-          <mesh filename="package://gimbalrotor/urdf/quad/mesh/rotor_arm.STL"/>
+          <mesh filename="package://gimbalrotor/urdf/quad/mesh/rotor_arm.stl"/>
         </geometry>
       </visual>
@@ -128,5 +128,5 @@
         <origin xyz="0 0 0" rpy="0 0 0"/>
         <geometry>
-          <mesh filename="package://gimbalrotor/urdf/quad/mesh/rotor_arm.STL"/>
+          <mesh filename="package://gimbalrotor/urdf/quad/mesh/rotor_arm.stl"/>
         </geometry>
       </visual>
@@ -156,5 +156,5 @@
         <origin xyz="0 0 0" rpy="0 0 0"/>
         <geometry>
-          <mesh filename="package://gimbalrotor/urdf/quad/mesh/rotor_arm.STL"/>
+          <mesh filename="package://gimbalrotor/urdf/quad/mesh/rotor_arm.stl"/>
         </geometry>
       </visual>
@@ -194,5 +194,5 @@
         <origin xyz="0 0 0" rpy="0 0 0"/>
         <geometry>
-          <mesh filename="package://gimbalrotor/urdf/quad/mesh/rotor_module.STL"/>
+          <mesh filename="package://gimbalrotor/urdf/quad/mesh/rotor_module.stl"/>
         </geometry>
       </visual>
@@ -216,7 +216,7 @@
         <mass value="0.00001"/>
         <inertia
-            ixx="0.001" ixy="0.0" ixz="0.0"
-            iyy="0.001" iyz="0.0"
-            izz="0.001"/>
+            ixx="0.000001" ixy="0.0" ixz="0.0"
+            iyy="0.000001" iyz="0.0"
+            izz="0.000001"/>
       </inertial>
     </link>
@@ -232,4 +232,8 @@
       <dynamics damping="0.8" friction="0.0"/>
     </joint>
+    <!-- This prevents NaN in Gazebo when virtual link inertia is too small -->
+    <gazebo reference="gimbal${self}">
+      <implicitSpringDamper>true</implicitSpringDamper>
+    </gazebo>
     <transmission name="joint_tran${self}">
       <type>transmission_interface/SimpleTransmission</type>

File: robots/gimbalrotor/urdf/ynltilt/gimbalrotor.urdf.xacro (robot description, xacro)
@@ -186,4 +186,8 @@
       <dynamics damping="0.8" friction="0.0"/>
     </joint>
+    <!-- This prevents NaN in Gazebo when virtual link inertia is too small -->
+    <gazebo reference="gimbal${self}">
+      <implicitSpringDamper>true</implicitSpringDamper>
+    </gazebo>
     <transmission name="joint_tran${self}">
       <type>transmission_interface/SimpleTransmission</type>
